Commit message: Updating

File: bartender_description/model/glass.urdf.xacro (robot description, xacro)
@@ -7,11 +7,11 @@
 <xacro:property name="gr_to_Kg" value="0.001"/>
 <!-- not so negligible, otherwise simulation fails -->
-<xacro:property name="bottle_mass" value="${1000*gr_to_Kg}"/>
-<xacro:property name="bottle_inertia">
+<xacro:property name="glass_mass" value="${200*gr_to_Kg}"/>
+<xacro:property name="glass_inertia">
     	<origin xyz="0 0 0"/>
-    	<mass value="${bottle_mass}"/>
-    	<inertia ixx="${bottle_mass * 10 * mm2_to_m2}" ixy="0.0" ixz="0.0" iyy="${bottle_mass * 10 * mm2_to_m2}" iyz="0.0" izz="${bottle_mass * 10 * mm2_to_m2}"/>
+    	<mass value="${glass_mass}"/>
+    	<inertia ixx="${glass_mass * 10 * mm2_to_m2}" ixy="0.0" ixz="0.0" iyy="${glass_mass * 10 * mm2_to_m2}" iyz="0.0" izz="${glass_mass * 10 * mm2_to_m2}"/>
 </xacro:property>
-<xacro:macro name="model_bottle" params="parent name *origin **material">
+<xacro:macro name="model_glass" params="parent name *origin">
   	<joint name="${parent}_${name}_base_joint" type="fixed">
     		<insert_block name="origin"/>
@@ -20,18 +20,18 @@
   	</joint>
   	<link name="${name}_link">
-      <insert_block name="material"/>
     		<inertial>
-      			<insert_block name="bottle_inertia"/>
+      			<insert_block name="glass_inertia"/>
     		</inertial>
     		<visual>
 			<origin xyz="0 0 0" rpy="0 0 0"/>
 			<geometry>
-				<cylinder length="0.3" radius="0.05"/>
+				<cylinder length="0.15" radius="0.05"/>
 			</geometry>
+      <material name="Vito/Silver"/>
     		</visual>
 		<collision>
 			<origin xyz="0 0 0" rpy="0 0 0"/>
 			<geometry>
-				<cylinder length="0.3" radius="0.05"/>
+				<cylinder length="0.15" radius="0.05"/>
 			</geometry>
 		</collision>

File: bartender_description/robot/bartender.urdf.xacro (robot description, xacro)
@@ -9,4 +9,5 @@
   <xacro:include filename="$(find soft_hand_description)/model/soft_hand.urdf.xacro"/>
   <xacro:include filename="$(find bartender_description)/model/bottle.urdf.xacro"/>
+  <xacro:include filename="$(find bartender_description)/model/glass.urdf.xacro"/>
   <link name="bartender_anchor" />
    <link name="world"/>
@@ -36,11 +37,18 @@
   <xacro:model_bottle name="bottle_R" parent="bartender_anchor">
     <origin xyz="-1.0 0 0.22" rpy="0 0 0"/>
+    <material name="Vito/Blue"/>
   </xacro:model_bottle>
   <xacro:model_bottle name="bottle_B" parent="bartender_anchor">
     <origin xyz="-1.0 0.3 0.22" rpy="0 0 0"/>
+    <material name="Vito/LightGrey"/>
   </xacro:model_bottle>
   <xacro:model_bottle name="bottle_O" parent="bartender_anchor">
     <origin xyz="-1.0 -0.3 0.22" rpy="0 0 0"/>
+    <material name="Vito/Orange"/>
   </xacro:model_bottle>
+  <!-- GLASS -->
+  <xacro:model_glass name="glass_drink" parent="bartender_anchor">
+    <origin xyz="-0.7 0 0.15" rpy="0 0 0"/>
+  </xacro:model_glass>
   <!-- TORSO -->
   <xacro:model_torso name="torso" parent="bartender_anchor">
@@ -52,7 +60,7 @@
   </xacro:kuka_lwr>
   <!-- LEFT SOFTHAND -->
-  <!-- xacro:soft_hand parent="left_arm_7_link" name="left_hand" left="true" withAdaptiveTransmission="true" useMimicTag="true">
+  <!-- <xacro:soft_hand parent="left_arm_7_link" name="left_hand" left="true" withAdaptiveTransmission="true" useMimicTag="true">
     <origin xyz="0 0 0" rpy="0 0 0"/>
-  </xacro:soft_hand -->
+  </xacro:soft_hand > -->
   <!-- RIGHT ARM -->
   <xacro:kuka_lwr name="right_arm" parent="bartender_anchor">
@@ -60,6 +68,6 @@
   </xacro:kuka_lwr>
   <!-- RIGHT SOFTHAND -->
-  <!-- xacro:soft_hand parent="right_arm_7_link" name="right_hand" left="false" withAdaptiveTransmission="true" useMimicTag="true">
+  <!-- <xacro:soft_hand parent="right_arm_7_link" name="right_hand" left="false" withAdaptiveTransmission="true" useMimicTag="true">
     <origin xyz="0 0 0" rpy="0 0 0"/>
-  </xacro:soft_hand -->
+  </xacro:soft_hand > -->
 </robot>

File: bartender_description/robot/environment.urdf.xacro (robot description, xacro)
@@ -4,6 +4,7 @@
   <!-- MODELS -->
   <xacro:include filename="$(find bartender_description)/model/table.urdf.xacro"/>
-  <xacro:include filename="$(find bartender_description)/model/materials.urdf"/>
+  <xacro:include filename="$(find vito_description)/model/materials.urdf"/>
   <xacro:include filename="$(find bartender_description)/model/bottle.xacro"/>
+<xacro:include filename="$(find bartender_description)/model/glass.xacro"/>
   <!-- WORKBENCH -->
   <link name="bartender_workbench_anchor"/>
