Commit message: added new bootles, function param_update in control.cpp

File: bartender_description/model/bottle.urdf.xacro (robot description, xacro)
@@ -27,5 +27,5 @@
 			<origin xyz="0 0 0" rpy="0 0 0"/>
 			<geometry>
-				<cylinder length="0.3" radius="0.05"/>
+				<cylinder length="0.3" radius="0.03"/>
 			</geometry>
     		</visual>
@@ -33,5 +33,5 @@
 			<origin xyz="0 0 0" rpy="0 0 0"/>
 			<geometry>
-				<cylinder length="0.3" radius="0.05"/>
+				<cylinder length="0.3" radius="0.03"/>
 			</geometry>
 		</collision>

File: bartender_description/robot/bartender.urdf.xacro (robot description, xacro)
@@ -40,10 +40,18 @@
   </xacro:model_bottle>
   <xacro:model_bottle name="bottle_B" parent="bartender_anchor">
-    <origin xyz="-1.0 0.3 0.22" rpy="0 0 0"/>
+    <origin xyz="-1.0 0.2 0.22" rpy="0 0 0"/>
     <material name="Vito/LightGrey"/>
   </xacro:model_bottle>
   <xacro:model_bottle name="bottle_O" parent="bartender_anchor">
-    <origin xyz="-1.0 -0.3 0.22" rpy="0 0 0"/>
+    <origin xyz="-1.0 -0.2 0.22" rpy="0 0 0"/>
     <material name="Vito/Orange"/>
+  </xacro:model_bottle>
+  <xacro:model_bottle name="bottle_G" parent="bartender_anchor">
+    <origin xyz="-1.0 0.4 0.22" rpy="0 0 0"/>
+    <material name="Vito/Green"/>
+  </xacro:model_bottle>
+  <xacro:model_bottle name="bottle_Y" parent="bartender_anchor">
+    <origin xyz="-1.0 -0.4 0.22" rpy="0 0 0"/>
+    <material name="Vito/Yellow"/>
   </xacro:model_bottle>
   <!-- GLASS -->
