Commit message: finishing message from manager to controller

File: bartender_description/robot/bartender.urdf.xacro (robot description, xacro)
@@ -73,9 +73,9 @@
   <!-- RIGHT ARM -->
   <xacro:kuka_lwr name="right_arm" parent="bartender_anchor">
-    <origin xyz="-0.165 0.10858 0.390" rpy="-1.5707963267948966 0.5235987010713441 0.5235990737060282"/>
+    <origin xyz="-0.165 0.10858 0.390" rpy="-1.5707963267948966 -0.5235987010713441 0.5235990737060282"/>
   </xacro:kuka_lwr>
   <!-- RIGHT SOFTHAND -->
   <xacro:soft_hand parent="right_arm_7_link" name="right_hand" left="false" withAdaptiveTransmission="true" useMimicTag="true">
-    <origin xyz="0 0 0" rpy="0 0 0"/>
+    <origin xyz="0 0 0" rpy="0 0 ${pi}"/>
   </xacro:soft_hand >
 </robot>
